Commit message: feat: integrate CAD-derived Poppy Ergo Jr arm

File: results/verified/diagnostic/robot.urdf (robot description, URDF)
Before this commit: robot mobile_manipulator, 13 links, 12 joints
Links:
- removed link forearm_link
- removed link left_finger
- removed link right_finger
- removed link shoulder_link
- removed link upper_arm_link
- removed link wrist_link
- added link poppy_link_1, mass 0.0223; collision box size=0.040 0.032 0.062; visual box size=0.024 0.027 0.036
- added link poppy_link_2, mass 0.0216; collision box size=0.040 0.030 0.050; visual box size=0.027 0.024 0.036
- added link poppy_link_3, mass 0.0186; collision box size=0.036 0.032 0.060; visual box size=0.024 0.027 0.036
- added link poppy_link_4, mass 0.0216; collision box size=0.040 0.030 0.050; visual box size=0.027 0.024 0.036
- added link poppy_link_5, mass 0.0244; collision box size=0.024 0.032 0.028; collision box size=0.092 0.008 0.024
- added link poppy_link_6, mass 0.00614; collision mesh filename=file:///home/dryanguasr/proyectos/gazebo-tutorial/gazebo-co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; visual mesh filename=file:///home/dryanguasr/proyectos/gazebo-tutorial/gazebo-co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
- added link poppy_mount_link, mass 0.0283; collision mesh filename=file:///home/dryanguasr/proyectos/gazebo-tutorial/gazebo-co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; visual box size=0.024 0.027 0.036
Joints:
- removed joint arm_base_yaw
- removed joint elbow_pitch
- removed joint left_finger_joint
- removed joint right_finger_joint
- removed joint shoulder_pitch
- removed joint wrist_pitch
- added joint poppy_m1_joint: type revolute, parent poppy_mount_link, child poppy_link_1, origin xyz=0 0 0.0328, axis 0 0 1, limit lower=-2.61799 upper=2.61799 effort=0.39 velocity=2.0
- added joint poppy_m2_joint: type revolute, parent poppy_link_1, child poppy_link_2, origin xyz=0 0 0.024, axis 0 1 0, limit lower=-1.5708 upper=1.5708 effort=0.39 velocity=2.0
- added joint poppy_m3_joint: type revolute, parent poppy_link_2, child poppy_link_3, origin xyz=0 0 0.054, axis 1 0 0, limit lower=-1.5708 upper=1.5708 effort=0.39 velocity=2.0
- added joint poppy_m4_joint: type revolute, parent poppy_link_3, child poppy_link_4, origin xyz=0 0 0.045, axis 0 1 0, limit lower=-1.5708 upper=1.5708 effort=0.39 velocity=2.0
- added joint poppy_m5_joint: type revolute, parent poppy_link_4, child poppy_link_5, origin xyz=0 0 0.048, axis 1 0 0, limit lower=-1.5708 upper=1.5708 effort=0.39 velocity=2.0
- added joint poppy_m6_joint: type revolute, parent poppy_link_5, child poppy_link_6, origin xyz=0 0 0.058, axis 0 1 0, limit lower=0.0 upper=1.20 effort=0.39 velocity=2.0
- added joint poppy_mount_joint: type fixed, parent base_link, child poppy_mount_link, origin xyz=-0.05 0 0.08
- joint front_left_joint: limit (none) -> effort=40 velocity=12.0
- joint front_right_joint: limit (none) -> effort=40 velocity=12.0
- joint rear_left_joint: limit (none) -> effort=40 velocity=12.0
- joint rear_right_joint: limit (none) -> effort=40 velocity=12.0

File: src/mobile_manipulator/urdf/mobile_manipulator.urdf.xacro (robot description, xacro)
@@ -3,30 +3,340 @@
   <material name="SlateGray"><color rgba="0.44 0.50 0.56 1"/></material>
   <material name="Black"><color rgba="0.04 0.04 0.04 1"/></material>
-  <material name="DarkOrange"><color rgba="1.0 0.35 0.0 1"/></material>
-  <material name="Goldenrod"><color rgba="0.85 0.65 0.13 1"/></material>
-  <material name="Khaki"><color rgba="0.94 0.90 0.55 1"/></material>
-  <material name="LightSteelBlue"><color rgba="0.69 0.77 0.87 1"/></material>
-  <material name="Silver"><color rgba="0.75 0.75 0.75 1"/></material>
+  <material name="PoppyOrange"><color rgba="1.0 0.32 0.05 1"/></material>
+  <material name="ServoGray"><color rgba="0.28 0.30 0.32 1"/></material>
   <material name="Blue"><color rgba="0.1 0.25 0.9 1"/></material>
   <xacro:macro name="box" params="name xyz size mass color">
-    <link name="${name}"><inertial><mass value="${mass}"/><inertia ixx="0.01" iyy="0.01" izz="0.01" ixy="0" ixz="0" iyz="0"/></inertial><visual><origin xyz="${xyz}"/><geometry><box size="${size}"/></geometry><material name="${color}"/></visual><collision><origin xyz="${xyz}"/><geometry><box size="${size}"/></geometry></collision></link>
+    <link name="${name}">
+      <inertial>
+        <mass value="${mass}"/>
+        <inertia ixx="0.01" iyy="0.01" izz="0.01" ixy="0" ixz="0" iyz="0"/>
+      </inertial>
+      <visual>
+        <origin xyz="${xyz}"/>
+        <geometry><box size="${size}"/></geometry>
+        <material name="${color}"/>
+      </visual>
+      <collision>
+        <origin xyz="${xyz}"/>
+        <geometry><box size="${size}"/></geometry>
+      </collision>
+    </link>
   </xacro:macro>
   <xacro:box name="base_link" xyz="0 0 0" size="0.72 0.52 0.16" mass="18" color="SlateGray"/>
-  <link name="base_footprint"/><joint name="base_fixed" type="fixed"><parent link="base_footprint"/><child link="base_link"/><origin xyz="0 0 0.16"/></joint>
-  <xacro:macro name="wheel" params="name x y"><link name="${name}_link"><inertial><mass value="1.2"/><inertia ixx="0.006" iyy="0.006" izz="0.01" ixy="0" ixz="0" iyz="0"/></inertial><visual><origin rpy="1.5708 0 0"/><geometry><cylinder radius="0.115" length="0.07"/></geometry><material name="Black"/></visual><collision><origin rpy="1.5708 0 0"/><geometry><cylinder radius="0.115" length="0.07"/></geometry></collision></link><joint name="${name}_joint" type="continuous"><parent link="base_link"/><child link="${name}_link"/><origin xyz="${x} ${y} 0"/><axis xyz="0 1 0"/><limit effort="40" velocity="12.0"/></joint></xacro:macro>
-  <xacro:wheel name="front_left" x="0.25" y="0.30"/><xacro:wheel name="rear_left" x="-0.25" y="0.30"/><xacro:wheel name="front_right" x="0.25" y="-0.30"/><xacro:wheel name="rear_right" x="-0.25" y="-0.30"/>
-  <xacro:box name="shoulder_link" xyz="0 0 0.13" size="0.18 0.18 0.26" mass="3" color="DarkOrange"/>
-  <joint name="arm_base_yaw" type="revolute"><parent link="base_link"/><child link="shoulder_link"/><origin xyz="-0.05 0 0.08"/><axis xyz="0 0 1"/><limit lower="-3.14" upper="3.14" effort="30" velocity="1.5"/></joint>
-  <xacro:box name="upper_arm_link" xyz="0.17 0 0" size="0.34 0.14 0.14" mass="2.2" color="Goldenrod"/>
-  <joint name="shoulder_pitch" type="revolute"><parent link="shoulder_link"/><child link="upper_arm_link"/><origin xyz="0 0 0.22"/><axis xyz="0 1 0"/><limit lower="-1.5" upper="1.5" effort="25" velocity="1.5"/></joint>
-  <xacro:box name="forearm_link" xyz="0.15 0 0" size="0.30 0.12 0.12" mass="1.5" color="Khaki"/>
-  <joint name="elbow_pitch" type="revolute"><parent link="upper_arm_link"/><child link="forearm_link"/><origin xyz="0.34 0 0"/><axis xyz="0 1 0"/><limit lower="-2.0" upper="2.0" effort="20" velocity="1.8"/></joint>
-  <xacro:box name="wrist_link" xyz="0.10 0 0" size="0.20 0.10 0.10" mass="0.8" color="LightSteelBlue"/>
-  <joint name="wrist_pitch" type="revolute"><parent link="forearm_link"/><child link="wrist_link"/><origin xyz="0.30 0 0"/><axis xyz="0 1 0"/><limit lower="-1.8" upper="1.8" effort="12" velocity="2.0"/></joint>
-  <xacro:box name="left_finger" xyz="0.15 0.045 0" size="0.16 0.035 0.07" mass="0.12" color="Silver"/><xacro:box name="right_finger" xyz="0.15 -0.045 0" size="0.16 0.035 0.07" mass="0.12" color="Silver"/>
-  <joint name="left_finger_joint" type="prismatic"><parent link="wrist_link"/><child link="left_finger"/><origin xyz="0.20 0.045 0"/><axis xyz="0 1 0"/><limit lower="0" upper="0.04" effort="8" velocity="0.1"/></joint><joint name="right_finger_joint" type="prismatic"><parent link="wrist_link"/><child link="right_finger"/><origin xyz="0.20 -0.045 0"/><axis xyz="0 1 0"/><limit lower="-0.04" upper="0" effort="8" velocity="0.1"/></joint>
-  <link name="camera_link"><visual><geometry><box size="0.08 0.12 0.06"/></geometry><material name="Blue"/></visual></link><joint name="camera_fixed" type="fixed"><parent link="base_link"/><child link="camera_link"/><origin xyz="0.38 0 0.10" rpy="0 0 0"/></joint>
-  <ros2_control name="GazeboSimSystem" type="system"><hardware><plugin>gz_ros2_control/GazeboSimSystem</plugin></hardware><joint name="front_left_joint"><command_interface name="velocity"/><state_interface name="position"/><state_interface name="velocity"/></joint><joint name="rear_left_joint"><command_interface name="velocity"/><state_interface name="position"/><state_interface name="velocity"/></joint><joint name="front_right_joint"><command_interface name="velocity"/><state_interface name="position"/><state_interface name="velocity"/></joint><joint name="rear_right_joint"><command_interface name="velocity"/><state_interface name="position"/><state_interface name="velocity"/></joint><joint name="arm_base_yaw"><command_interface name="position"/><state_interface name="position"/></joint><joint name="shoulder_pitch"><command_interface name="position"/><state_interface name="position"/></joint><joint name="elbow_pitch"><command_interface name="position"/><state_interface name="position"/></joint><joint name="wrist_pitch"><command_interface name="position"/><state_interface name="position"/></joint><joint name="left_finger_joint"><command_interface name="position"/><state_interface name="position"/></joint><joint name="right_finger_joint"><command_interface name="position"/><state_interface name="position"/></joint></ros2_control>
-  <gazebo reference="camera_link"><sensor name="front_camera" type="camera"><topic>/camera/image_raw</topic><update_rate>30</update_rate><camera><horizontal_fov>1.047</horizontal_fov><image><width>640</width><height>480</height><format>R8G8B8</format></image><clip><near>0.05</near><far>20</far></clip></camera></sensor></gazebo>
-  <gazebo><plugin filename="gz_ros2_control-system" name="gz_ros2_control::GazeboSimROS2ControlPlugin"><parameters>$(find mobile_manipulator)/config/controllers.yaml</parameters></plugin></gazebo>
+  <link name="base_footprint"/>
+  <joint name="base_fixed" type="fixed">
+    <parent link="base_footprint"/>
+    <child link="base_link"/>
+    <origin xyz="0 0 0.16"/>
+  </joint>
+  <xacro:macro name="wheel" params="name x y">
+    <link name="${name}_link">
+      <inertial>
+        <mass value="1.2"/>
+        <inertia ixx="0.006" iyy="0.006" izz="0.01" ixy="0" ixz="0" iyz="0"/>
+      </inertial>
+      <visual>
+        <origin rpy="1.5708 0 0"/>
+        <geometry><cylinder radius="0.115" length="0.07"/></geometry>
+        <material name="Black"/>
+      </visual>
+      <collision>
+        <origin rpy="1.5708 0 0"/>
+        <geometry><cylinder radius="0.115" length="0.07"/></geometry>
+      </collision>
+    </link>
+    <joint name="${name}_joint" type="continuous">
+      <parent link="base_link"/>
+      <child link="${name}_link"/>
+      <origin xyz="${x} ${y} 0"/>
+      <axis xyz="0 1 0"/>
+      <limit effort="40" velocity="12.0"/>
+    </joint>
+  </xacro:macro>
+  <xacro:wheel name="front_left" x="0.25" y="0.30"/>
+  <xacro:wheel name="rear_left" x="-0.25" y="0.30"/>
+  <xacro:wheel name="front_right" x="0.25" y="-0.30"/>
+  <xacro:wheel name="rear_right" x="-0.25" y="-0.30"/>
+  <!-- The printed Poppy base and motor m1 body remain fixed to the vehicle. -->
+  <link name="poppy_mount_link">
+    <inertial>
+      <origin xyz="0 0 0.025"/>
+      <mass value="0.0283"/>
+      <inertia ixx="1.36e-5" iyy="1.36e-5" izz="1.53e-5" ixy="0" ixz="0" iyz="0"/>
+    </inertial>
+    <visual>
+      <geometry>
+        <mesh filename="file://$(find mobile_manipulator)/meshes/poppy_ergo_jr/visual/poppy_mount.stl"/>
+      </geometry>
+      <material name="PoppyOrange"/>
+    </visual>
+    <visual>
+      <origin xyz="0 0 0.027"/>
+      <geometry><box size="0.024 0.027 0.036"/></geometry>
+      <material name="ServoGray"/>
+    </visual>
+    <collision>
+      <geometry>
+        <mesh filename="file://$(find mobile_manipulator)/meshes/poppy_ergo_jr/collision/poppy_mount_convex.stl"/>
+      </geometry>
+    </collision>
+  </link>
+  <joint name="poppy_mount_joint" type="fixed">
+    <parent link="base_link"/>
+    <child link="poppy_mount_link"/>
+    <origin xyz="-0.05 0 0.08"/>
+  </joint>
+  <link name="poppy_link_1">
+    <inertial>
+      <origin xyz="0 0 0.025"/>
+      <mass value="0.0223"/>
+      <inertia ixx="6.32e-6" iyy="7.62e-6" izz="4.65e-6" ixy="0" ixz="0" iyz="0"/>
+    </inertial>
+    <visual>
+      <geometry>
+        <mesh filename="file://$(find mobile_manipulator)/meshes/poppy_ergo_jr/visual/poppy_link_1.stl"/>
+      </geometry>
+      <material name="PoppyOrange"/>
+    </visual>
+    <visual>
+      <origin xyz="0 0 0.024"/>
+      <geometry><box size="0.024 0.027 0.036"/></geometry>
+      <material name="ServoGray"/>
+    </visual>
+    <collision>
+      <origin xyz="0 0 0.031"/>
+      <geometry><box size="0.040 0.032 0.062"/></geometry>
+    </collision>
+  </link>
+  <joint name="poppy_m1_joint" type="revolute">
+    <parent link="poppy_mount_link"/>
+    <child link="poppy_link_1"/>
+    <origin xyz="0 0 0.0328"/>
+    <axis xyz="0 0 1"/>
+    <limit lower="-2.61799" upper="2.61799" effort="0.39" velocity="2.0"/>
+  </joint>
+  <link name="poppy_link_2">
+    <inertial>
+      <origin xyz="0 0 0.041"/>
+      <mass value="0.0216"/>
+      <inertia ixx="8.99e-6" iyy="1.03e-5" izz="4.50e-6" ixy="0" ixz="0" iyz="0"/>
+    </inertial>
+    <visual>
+      <geometry>
+        <mesh filename="file://$(find mobile_manipulator)/meshes/poppy_ergo_jr/visual/poppy_link_2.stl"/>
+      </geometry>
+      <material name="PoppyOrange"/>
+    </visual>
+    <visual>
+      <origin xyz="0 0 0.054"/>
+      <geometry><box size="0.027 0.024 0.036"/></geometry>
+      <material name="ServoGray"/>
+    </visual>
+    <collision>
+      <origin xyz="0 0 0.0415"/>
+      <geometry><box size="0.040 0.030 0.050"/></geometry>
+    </collision>
+  </link>
+  <joint name="poppy_m2_joint" type="revolute">
+    <parent link="poppy_link_1"/>
+    <child link="poppy_link_2"/>
+    <origin xyz="0 0 0.024"/>
+    <axis xyz="0 1 0"/>
+    <limit lower="-1.5708" upper="1.5708" effort="0.39" velocity="2.0"/>
+  </joint>
+  <link name="poppy_link_3">
+    <inertial>
+      <origin xyz="0 0 0.030"/>
+      <mass value="0.0186"/>
+      <inertia ixx="6.98e-6" iyy="7.48e-6" izz="3.29e-6" ixy="0" ixz="0" iyz="0"/>
+    </inertial>
+    <visual>
+      <geometry>
+        <mesh filename="file://$(find mobile_manipulator)/meshes/poppy_ergo_jr/visual/poppy_link_3.stl"/>
+      </geometry>
+      <material name="PoppyOrange"/>
+    </visual>
+    <visual>
+      <origin xyz="0 0 0.045"/>
+      <geometry><box size="0.024 0.027 0.036"/></geometry>
+      <material name="ServoGray"/>
+    </visual>
+    <collision>
+      <origin xyz="0 0 0.030"/>
+      <geometry><box size="0.036 0.032 0.060"/></geometry>
+    </collision>
+  </link>
+  <joint name="poppy_m3_joint" type="revolute">
+    <parent link="poppy_link_2"/>
+    <child link="poppy_link_3"/>
+    <origin xyz="0 0 0.054"/>
+    <axis xyz="1 0 0"/>
+    <limit lower="-1.5708" upper="1.5708" effort="0.39" velocity="2.0"/>
+  </joint>
+  <link name="poppy_link_4">
+    <inertial>
+      <origin xyz="0 0 0.041"/>
+      <mass value="0.0216"/>
+      <inertia ixx="8.99e-6" iyy="1.03e-5" izz="4.50e-6" ixy="0" ixz="0" iyz="0"/>
+    </inertial>
+    <visual>
+      <geometry>
+        <mesh filename="file://$(find mobile_manipulator)/meshes/poppy_ergo_jr/visual/poppy_link_4.stl"/>
+      </geometry>
+      <material name="PoppyOrange"/>
+    </visual>
+    <visual>
+      <origin xyz="0 0 0.048"/>
+      <geometry><box size="0.027 0.024 0.036"/></geometry>
+      <material name="ServoGray"/>
+    </visual>
+    <collision>
+      <origin xyz="0 0 0.0415"/>
+      <geometry><box size="0.040 0.030 0.050"/></geometry>
+    </collision>
+  </link>
+  <joint name="poppy_m4_joint" type="revolute">
+    <parent link="poppy_link_3"/>
+    <child link="poppy_link_4"/>
+    <origin xyz="0 0 0.045"/>
+    <axis xyz="0 1 0"/>
+    <limit lower="-1.5708" upper="1.5708" effort="0.39" velocity="2.0"/>
+  </joint>
+  <link name="poppy_link_5">
+    <inertial>
+      <origin xyz="0.025 0 0.045"/>
+      <mass value="0.0244"/>
+      <inertia ixx="1.06e-5" iyy="2.77e-5" izz="2.36e-5" ixy="0" ixz="0" iyz="0"/>
+    </inertial>
+    <visual>
+      <geometry>
+        <mesh filename="file://$(find mobile_manipulator)/meshes/poppy_ergo_jr/visual/poppy_link_5.stl"/>
+      </geometry>
+      <material name="PoppyOrange"/>
+    </visual>
+    <visual>
+      <origin xyz="0 0 0.058"/>
+      <geometry><box size="0.024 0.027 0.036"/></geometry>
+      <material name="ServoGray"/>
+    </visual>
+    <collision>
+      <origin xyz="0 0 0.032"/>
+      <geometry><box size="0.024 0.032 0.028"/></geometry>
+    </collision>
+    <collision>
+      <origin xyz="0.025 0.0145 0.058"/>
+      <geometry><box size="0.092 0.008 0.024"/></geometry>
+    </collision>
+  </link>
+  <joint name="poppy_m5_joint" type="revolute">
+    <parent link="poppy_link_4"/>
+    <child link="poppy_link_5"/>
+    <origin xyz="0 0 0.048"/>
+    <axis xyz="1 0 0"/>
+    <limit lower="-1.5708" upper="1.5708" effort="0.39" velocity="2.0"/>
+  </joint>
+  <link name="poppy_link_6">
+    <inertial>
+      <origin xyz="0.030 -0.0035 0"/>
+      <mass value="0.00614"/>
+      <inertia ixx="9.72e-7" iyy="3.87e-6" izz="3.65e-6" ixy="0" ixz="0" iyz="0"/>
+    </inertial>
+    <visual>
+      <geometry>
+        <mesh filename="file://$(find mobile_manipulator)/meshes/poppy_ergo_jr/visual/poppy_link_6.stl"/>
+      </geometry>
+      <material name="PoppyOrange"/>
+    </visual>
+    <collision>
+      <geometry>
+        <mesh filename="file://$(find mobile_manipulator)/meshes/poppy_ergo_jr/collision/poppy_link_6_convex.stl"/>
+      </geometry>
+    </collision>
+  </link>
+  <joint name="poppy_m6_joint" type="revolute">
+    <parent link="poppy_link_5"/>
+    <child link="poppy_link_6"/>
+    <origin xyz="0 0 0.058"/>
+    <axis xyz="0 1 0"/>
+    <limit lower="0.0" upper="1.20" effort="0.39" velocity="2.0"/>
+  </joint>
+  <!-- The tracking camera stays on the vehicle front to preserve the A/B task. -->
+  <link name="camera_link">
+    <visual>
+      <geometry><box size="0.08 0.12 0.06"/></geometry>
+      <material name="Blue"/>
+    </visual>
+  </link>
+  <joint name="camera_fixed" type="fixed">
+    <parent link="base_link"/>
+    <child link="camera_link"/>
+    <origin xyz="0.38 0 0.10" rpy="0 0 0"/>
+  </joint>
+  <ros2_control name="GazeboSimSystem" type="system">
+    <hardware><plugin>gz_ros2_control/GazeboSimSystem</plugin></hardware>
+    <joint name="front_left_joint">
+      <command_interface name="velocity"/>
+      <state_interface name="position"/>
+      <state_interface name="velocity"/>
+    </joint>
+    <joint name="rear_left_joint">
+      <command_interface name="velocity"/>
+      <state_interface name="position"/>
+      <state_interface name="velocity"/>
+    </joint>
+    <joint name="front_right_joint">
+      <command_interface name="velocity"/>
+      <state_interface name="position"/>
+      <state_interface name="velocity"/>
+    </joint>
+    <joint name="rear_right_joint">
+      <command_interface name="velocity"/>
+      <state_interface name="position"/>
+      <state_interface name="velocity"/>
+    </joint>
+    <joint name="poppy_m1_joint">
+      <command_interface name="position"/>
+      <state_interface name="position"/>
+    </joint>
+    <joint name="poppy_m2_joint">
+      <command_interface name="position"/>
+      <state_interface name="position"/>
+    </joint>
+    <joint name="poppy_m3_joint">
+      <command_interface name="position"/>
+      <state_interface name="position"/>
+    </joint>
+    <joint name="poppy_m4_joint">
+      <command_interface name="position"/>
+      <state_interface name="position"/>
+    </joint>
+    <joint name="poppy_m5_joint">
+      <command_interface name="position"/>
+      <state_interface name="position"/>
+    </joint>
+    <joint name="poppy_m6_joint">
+      <command_interface name="position"/>
+      <state_interface name="position"/>
+    </joint>
+  </ros2_control>
+  <gazebo reference="camera_link">
+    <sensor name="front_camera" type="camera">
+      <topic>/camera/image_raw</topic>
+      <update_rate>30</update_rate>
+      <camera>
+        <horizontal_fov>1.047</horizontal_fov>
+        <image>
+          <width>640</width>
+          <height>480</height>
+          <format>R8G8B8</format>
+        </image>
+        <clip><near>0.05</near><far>20</far></clip>
+      </camera>
+    </sensor>
+  </gazebo>
+  <gazebo>
+    <plugin filename="gz_ros2_control-system" name="gz_ros2_control::GazeboSimROS2ControlPlugin">
+      <parameters>$(find mobile_manipulator)/config/controllers.yaml</parameters>
+    </plugin>
+  </gazebo>
 </robot>
