Commit message: Fix Poppy mechanical assembly and compact platform

File: results/verified/diagnostic/robot.urdf (robot description, URDF)
Before this commit: robot mobile_manipulator, 14 links, 13 joints
Links:
- added link poppy_fixed_tip
- added link poppy_moving_tip
- link base_link: mass 18 -> 6.0; geometry collision box size=0.4 0.3 0.1; visual box size=0.4 0.3 0.1
- link front_left_link: mass 1.2 -> 0.45; geometry collision cylinder length=0.045 radius=0.07; visual cylinder length=0.045 radius=0.07
- link front_right_link: mass 1.2 -> 0.45; geometry collision cylinder length=0.045 radius=0.07; visual cylinder length=0.045 radius=0.07
- link poppy_link_1: mass 0.0223 -> 0.0390; geometry collision box size=0.042 0.034 0.054; visual box size=0.024 0.027 0.036
- link poppy_link_2: mass 0.0216 -> 0.0383; geometry collision box size=0.050 0.030 0.040; visual box size=0.027 0.024 0.036
- link poppy_link_3: mass 0.0186 -> 0.0353; geometry collision box size=0.040 0.032 0.036; visual box size=0.024 0.027 0.036
- link poppy_link_4: mass 0.0216 -> 0.0383; geometry collision box size=0.040 0.050 0.030; visual box size=0.027 0.024 0.036
- link poppy_link_5: mass 0.0244 -> 0.0411; geometry collision box size=0.024 0.092 0.006; collision box size=0.036 0.032 0.030
- link poppy_mount_link: mass 0.0283 -> 0.0450
- link rear_left_link: mass 1.2 -> 0.45; geometry collision cylinder length=0.045 radius=0.07; visual cylinder length=0.045 radius=0.07
- link rear_right_link: mass 1.2 -> 0.45; geometry collision cylinder length=0.045 radius=0.07; visual cylinder length=0.045 radius=0.07
Joints:
- added joint poppy_fixed_tip_joint: type fixed, parent poppy_link_5, child poppy_fixed_tip, origin xyz=0 -0.11 0 rpy=-1.5707963267949 0 0
- added joint poppy_moving_tip_joint: type fixed, parent poppy_link_6, child poppy_moving_tip, origin xyz=0 -0.052 0 rpy=-1.5707963267949 0 0
- joint base_fixed: origin xyz=0 0 0.16 -> xyz=0 0 0.07
- joint camera_fixed: origin xyz=0.38 0 0.10 rpy=0 0 0 -> xyz=0.225 0 0.05 rpy=0 0 0
- joint front_left_joint: limit effort=40 velocity=12.0 -> effort=20 velocity=12.0; origin xyz=0.25 0.3 0 -> xyz=0.14 0.1725 0
- joint front_right_joint: limit effort=40 velocity=12.0 -> effort=20 velocity=12.0; origin xyz=0.25 -0.3 0 -> xyz=0.14 -0.1725 0
- joint poppy_m1_joint: origin xyz=0 0 0.0328 -> xyz=0 0 0.0327993216120967 rpy=0 0 0
- joint poppy_m2_joint: axis 0 1 0 -> 0 0 -1; origin xyz=0 0 0.024 -> xyz=0 0 0.0240006783879033 rpy=0 -1.5707963267949 0
- joint poppy_m3_joint: axis 1 0 0 -> 0 0 -1; origin xyz=0 0 0.054 -> xyz=0.054 0 0 rpy=0 0 0
- joint poppy_m4_joint: axis 0 1 0 -> 0 0 -1; origin xyz=0 0 0.045 -> xyz=0.045 0 0 rpy=0 -1.5707963267949 0
- joint poppy_m5_joint: axis 1 0 0 -> 0 0 1; origin xyz=0 0 0.048 -> xyz=0 -0.048 0 rpy=0 -1.5707963267949 0
- joint poppy_m6_joint: axis 0 1 0 -> 0 0 -1; origin xyz=0 0 0.058 -> xyz=0 -0.058 0 rpy=0 -1.5707963267949 0
- joint poppy_mount_joint: origin xyz=-0.05 0 0.08 -> xyz=-0.03 0 0.05
- joint rear_left_joint: limit effort=40 velocity=12.0 -> effort=20 velocity=12.0; origin xyz=-0.25 0.3 0 -> xyz=-0.14 0.1725 0
- joint rear_right_joint: limit effort=40 velocity=12.0 -> effort=20 velocity=12.0; origin xyz=-0.25 -0.3 0 -> xyz=-0.14 -0.1725 0

File: src/mobile_manipulator/urdf/mobile_manipulator.urdf.xacro (robot description, xacro)
@@ -6,9 +6,29 @@
   <material name="ServoGray"><color rgba="0.28 0.30 0.32 1"/></material>
   <material name="Blue"><color rgba="0.1 0.25 0.9 1"/></material>
-  <xacro:macro name="box" params="name xyz size mass color">
+  <!-- Compact platform selected after validating the Poppy CAD at physical 1:1. -->
+  <xacro:property name="base_length" value="0.40"/>
+  <xacro:property name="base_width" value="0.30"/>
+  <xacro:property name="base_height" value="0.10"/>
+  <xacro:property name="base_mass" value="6.0"/>
+  <xacro:property name="base_ixx" value="0.050"/>
+  <xacro:property name="base_iyy" value="0.085"/>
+  <xacro:property name="base_izz" value="0.125"/>
+  <xacro:property name="wheel_radius" value="0.070"/>
+  <xacro:property name="wheel_width" value="0.045"/>
+  <xacro:property name="wheel_mass" value="0.45"/>
+  <xacro:property name="wheel_ixx" value="0.000627"/>
+  <xacro:property name="wheel_iyy" value="0.001103"/>
+  <xacro:property name="wheel_izz" value="0.000627"/>
+  <xacro:property name="wheel_x" value="0.140"/>
+  <xacro:property name="wheel_y" value="0.1725"/>
+  <xacro:property name="camera_x" value="0.225"/>
+  <xacro:property name="camera_z" value="0.050"/>
+  <xacro:property name="arm_mount_x" value="-0.030"/>
+  <xacro:property name="arm_mount_z" value="0.050"/>
+  <xacro:macro name="box" params="name xyz size mass ixx iyy izz color">
     <link name="${name}">
       <inertial>
         <mass value="${mass}"/>
-        <inertia ixx="0.01" iyy="0.01" izz="0.01" ixy="0" ixz="0" iyz="0"/>
+        <inertia ixx="${ixx}" iyy="${iyy}" izz="${izz}" ixy="0" ixz="0" iyz="0"/>
       </inertial>
       <visual>
@@ -23,25 +43,34 @@
     </link>
   </xacro:macro>
-  <xacro:box name="base_link" xyz="0 0 0" size="0.72 0.52 0.16" mass="18" color="SlateGray"/>
+  <xacro:box
+    name="base_link"
+    xyz="0 0 0"
+    size="${base_length} ${base_width} ${base_height}"
+    mass="${base_mass}"
+    ixx="${base_ixx}"
+    iyy="${base_iyy}"
+    izz="${base_izz}"
+    color="SlateGray"
+  />
   <link name="base_footprint"/>
   <joint name="base_fixed" type="fixed">
     <parent link="base_footprint"/>
     <child link="base_link"/>
-    <origin xyz="0 0 0.16"/>
+    <origin xyz="0 0 ${wheel_radius}"/>
   </joint>
   <xacro:macro name="wheel" params="name x y">
     <link name="${name}_link">
       <inertial>
-        <mass value="1.2"/>
-        <inertia ixx="0.006" iyy="0.006" izz="0.01" ixy="0" ixz="0" iyz="0"/>
+        <mass value="${wheel_mass}"/>
+        <inertia ixx="${wheel_ixx}" iyy="${wheel_iyy}" izz="${wheel_izz}" ixy="0" ixz="0" iyz="0"/>
       </inertial>
       <visual>
-        <origin rpy="1.5708 0 0"/>
-        <geometry><cylinder radius="0.115" length="0.07"/></geometry>
+        <origin rpy="1.5707963267949 0 0"/>
+        <geometry><cylinder radius="${wheel_radius}" length="${wheel_width}"/></geometry>
         <material name="Black"/>
       </visual>
       <collision>
-        <origin rpy="1.5708 0 0"/>
-        <geometry><cylinder radius="0.115" length="0.07"/></geometry>
+        <origin rpy="1.5707963267949 0 0"/>
+        <geometry><cylinder radius="${wheel_radius}" length="${wheel_width}"/></geometry>
       </collision>
     </link>
@@ -51,17 +80,17 @@
       <origin xyz="${x} ${y} 0"/>
       <axis xyz="0 1 0"/>
-      <limit effort="40" velocity="12.0"/>
+      <limit effort="20" velocity="12.0"/>
     </joint>
   </xacro:macro>
-  <xacro:wheel name="front_left" x="0.25" y="0.30"/>
-  <xacro:wheel name="rear_left" x="-0.25" y="0.30"/>
-  <xacro:wheel name="front_right" x="0.25" y="-0.30"/>
-  <xacro:wheel name="rear_right" x="-0.25" y="-0.30"/>
+  <xacro:wheel name="front_left" x="${wheel_x}" y="${wheel_y}"/>
+  <xacro:wheel name="rear_left" x="-${wheel_x}" y="${wheel_y}"/>
+  <xacro:wheel name="front_right" x="${wheel_x}" y="-${wheel_y}"/>
+  <xacro:wheel name="rear_right" x="-${wheel_x}" y="-${wheel_y}"/>
   <!-- The printed Poppy base and motor m1 body remain fixed to the vehicle. -->
   <link name="poppy_mount_link">
     <inertial>
-      <origin xyz="0 0 0.025"/>
-      <mass value="0.0283"/>
-      <inertia ixx="1.36e-5" iyy="1.36e-5" izz="1.53e-5" ixy="0" ixz="0" iyz="0"/>
+      <origin xyz="0 0 0.019"/>
+      <mass value="0.0450"/>
+      <inertia ixx="1.4e-5" iyy="1.3e-5" izz="1.7e-5" ixy="0" ixz="0" iyz="0"/>
     </inertial>
     <visual>
@@ -85,11 +114,11 @@
     <parent link="base_link"/>
     <child link="poppy_mount_link"/>
-    <origin xyz="-0.05 0 0.08"/>
+    <origin xyz="${arm_mount_x} 0 ${arm_mount_z}"/>
   </joint>
   <link name="poppy_link_1">
     <inertial>
-      <origin xyz="0 0 0.025"/>
-      <mass value="0.0223"/>
-      <inertia ixx="6.32e-6" iyy="7.62e-6" izz="4.65e-6" ixy="0" ixz="0" iyz="0"/>
+      <origin xyz="0 0 0.024"/>
+      <mass value="0.0390"/>
+      <inertia ixx="8.6e-6" iyy="9.8e-6" izz="7.0e-6" ixy="0" ixz="0" iyz="0"/>
     </inertial>
     <visual>
@@ -105,6 +134,6 @@
     </visual>
     <collision>
-      <origin xyz="0 0 0.031"/>
-      <geometry><box size="0.040 0.032 0.062"/></geometry>
+      <origin xyz="0 0 0.027"/>
+      <geometry><box size="0.042 0.034 0.054"/></geometry>
     </collision>
   </link>
@@ -112,5 +141,5 @@
     <parent link="poppy_mount_link"/>
     <child link="poppy_link_1"/>
-    <origin xyz="0 0 0.0328"/>
+    <origin xyz="0 0 0.0327993216120967" rpy="0 0 0"/>
     <axis xyz="0 0 1"/>
     <limit lower="-2.61799" upper="2.61799" effort="0.39" velocity="2.0"/>
@@ -118,7 +147,7 @@
   <link name="poppy_link_2">
     <inertial>
-      <origin xyz="0 0 0.041"/>
-      <mass value="0.0216"/>
-      <inertia ixx="8.99e-6" iyy="1.03e-5" izz="4.50e-6" ixy="0" ixz="0" iyz="0"/>
+      <origin xyz="0.042 0 0"/>
+      <mass value="0.0383"/>
+      <inertia ixx="5.0e-6" iyy="9.0e-6" izz="8.0e-6" ixy="0" ixz="0" iyz="0"/>
     </inertial>
     <visual>
@@ -129,11 +158,11 @@
     </visual>
     <visual>
-      <origin xyz="0 0 0.054"/>
+      <origin xyz="0.054 0 0" rpy="0 1.5707963267949 0"/>
       <geometry><box size="0.027 0.024 0.036"/></geometry>
       <material name="ServoGray"/>
     </visual>
     <collision>
-      <origin xyz="0 0 0.0415"/>
-      <geometry><box size="0.040 0.030 0.050"/></geometry>
+      <origin xyz="0.0415 0 0"/>
+      <geometry><box size="0.050 0.030 0.040"/></geometry>
     </collision>
   </link>
@@ -141,13 +170,13 @@
     <parent link="poppy_link_1"/>
     <child link="poppy_link_2"/>
-    <origin xyz="0 0 0.024"/>
-    <axis xyz="0 1 0"/>
+    <origin xyz="0 0 0.0240006783879033" rpy="0 -1.5707963267949 0"/>
+    <axis xyz="0 0 -1"/>
     <limit lower="-1.5708" upper="1.5708" effort="0.39" velocity="2.0"/>
   </joint>
   <link name="poppy_link_3">
     <inertial>
-      <origin xyz="0 0 0.030"/>
-      <mass value="0.0186"/>
-      <inertia ixx="6.98e-6" iyy="7.48e-6" izz="3.29e-6" ixy="0" ixz="0" iyz="0"/>
+      <origin xyz="0.047 0 0"/>
+      <mass value="0.0353"/>
+      <inertia ixx="4.2e-6" iyy="5.0e-6" izz="4.5e-6" ixy="0" ixz="0" iyz="0"/>
     </inertial>
     <visual>
@@ -158,11 +187,11 @@
     </visual>
     <visual>
-      <origin xyz="0 0 0.045"/>
+      <origin xyz="0.045 0 0" rpy="0 1.5707963267949 0"/>
       <geometry><box size="0.024 0.027 0.036"/></geometry>
       <material name="ServoGray"/>
     </visual>
     <collision>
-      <origin xyz="0 0 0.030"/>
-      <geometry><box size="0.036 0.032 0.060"/></geometry>
+      <origin xyz="0.045 0 0"/>
+      <geometry><box size="0.040 0.032 0.036"/></geometry>
     </collision>
   </link>
@@ -170,13 +199,13 @@
     <parent link="poppy_link_2"/>
     <child link="poppy_link_3"/>
-    <origin xyz="0 0 0.054"/>
-    <axis xyz="1 0 0"/>
+    <origin xyz="0.054 0 0" rpy="0 0 0"/>
+    <axis xyz="0 0 -1"/>
     <limit lower="-1.5708" upper="1.5708" effort="0.39" velocity="2.0"/>
   </joint>
   <link name="poppy_link_4">
     <inertial>
-      <origin xyz="0 0 0.041"/>
-      <mass value="0.0216"/>
-      <inertia ixx="8.99e-6" iyy="1.03e-5" izz="4.50e-6" ixy="0" ixz="0" iyz="0"/>
+      <origin xyz="0 -0.042 0"/>
+      <mass value="0.0383"/>
+      <inertia ixx="9.0e-6" iyy="5.0e-6" izz="8.0e-6" ixy="0" ixz="0" iyz="0"/>
     </inertial>
     <visual>
@@ -187,11 +216,11 @@
     </visual>
     <visual>
-      <origin xyz="0 0 0.048"/>
+      <origin xyz="0 -0.048 0" rpy="1.5707963267949 0 0"/>
       <geometry><box size="0.027 0.024 0.036"/></geometry>
       <material name="ServoGray"/>
     </visual>
     <collision>
-      <origin xyz="0 0 0.0415"/>
-      <geometry><box size="0.040 0.030 0.050"/></geometry>
+      <origin xyz="0 -0.0415 0"/>
+      <geometry><box size="0.040 0.050 0.030"/></geometry>
     </collision>
   </link>
@@ -199,13 +228,13 @@
     <parent link="poppy_link_3"/>
     <child link="poppy_link_4"/>
-    <origin xyz="0 0 0.045"/>
-    <axis xyz="0 1 0"/>
+    <origin xyz="0.045 0 0" rpy="0 -1.5707963267949 0"/>
+    <axis xyz="0 0 -1"/>
     <limit lower="-1.5708" upper="1.5708" effort="0.39" velocity="2.0"/>
   </joint>
   <link name="poppy_link_5">
     <inertial>
-      <origin xyz="0.025 0 0.045"/>
-      <mass value="0.0244"/>
-      <inertia ixx="1.06e-5" iyy="2.77e-5" izz="2.36e-5" ixy="0" ixz="0" iyz="0"/>
+      <origin xyz="0 -0.070 0.005"/>
+      <mass value="0.0411"/>
+      <inertia ixx="4.7e-5" iyy="8.0e-6" izz="4.8e-5" ixy="0" ixz="0" iyz="0"/>
     </inertial>
     <visual>
@@ -216,15 +245,15 @@
     </visual>
     <visual>
-      <origin xyz="0 0 0.058"/>
+      <origin xyz="0 -0.058 0" rpy="0 -1.5707963267949 0"/>
       <geometry><box size="0.024 0.027 0.036"/></geometry>
       <material name="ServoGray"/>
     </visual>
     <collision>
-      <origin xyz="0 0 0.032"/>
-      <geometry><box size="0.024 0.032 0.028"/></geometry>
-    </collision>
-    <collision>
-      <origin xyz="0.025 0.0145 0.058"/>
-      <geometry><box size="0.092 0.008 0.024"/></geometry>
+      <origin xyz="0 -0.058 0"/>
+      <geometry><box size="0.036 0.032 0.030"/></geometry>
+    </collision>
+    <collision>
+      <origin xyz="0 -0.082 0.0145"/>
+      <geometry><box size="0.024 0.092 0.006"/></geometry>
     </collision>
   </link>
@@ -232,13 +261,13 @@
     <parent link="poppy_link_4"/>
     <child link="poppy_link_5"/>
-    <origin xyz="0 0 0.048"/>
-    <axis xyz="1 0 0"/>
+    <origin xyz="0 -0.048 0" rpy="0 -1.5707963267949 0"/>
+    <axis xyz="0 0 1"/>
     <limit lower="-1.5708" upper="1.5708" effort="0.39" velocity="2.0"/>
   </joint>
   <link name="poppy_link_6">
     <inertial>
-      <origin xyz="0.030 -0.0035 0"/>
+      <origin xyz="-0.0035 -0.030 0"/>
       <mass value="0.00614"/>
-      <inertia ixx="9.72e-7" iyy="3.87e-6" izz="3.65e-6" ixy="0" ixz="0" iyz="0"/>
+      <inertia ixx="3.87e-6" iyy="9.72e-7" izz="3.65e-6" ixy="0" ixz="0" iyz="0"/>
     </inertial>
     <visual>
@@ -257,7 +286,19 @@
     <parent link="poppy_link_5"/>
     <child link="poppy_link_6"/>
-    <origin xyz="0 0 0.058"/>
-    <axis xyz="0 1 0"/>
+    <origin xyz="0 -0.058 0" rpy="0 -1.5707963267949 0"/>
+    <axis xyz="0 0 -1"/>
     <limit lower="0.0" upper="1.20" effort="0.39" velocity="2.0"/>
+  </joint>
+  <link name="poppy_fixed_tip"/>
+  <joint name="poppy_fixed_tip_joint" type="fixed">
+    <parent link="poppy_link_5"/>
+    <child link="poppy_fixed_tip"/>
+    <origin xyz="0 -0.11 0" rpy="-1.5707963267949 0 0"/>
+  </joint>
+  <link name="poppy_moving_tip"/>
+  <joint name="poppy_moving_tip_joint" type="fixed">
+    <parent link="poppy_link_6"/>
+    <child link="poppy_moving_tip"/>
+    <origin xyz="0 -0.052 0" rpy="-1.5707963267949 0 0"/>
   </joint>
   <!-- The tracking camera stays on the vehicle front to preserve the A/B task. -->
@@ -271,5 +312,5 @@
     <parent link="base_link"/>
     <child link="camera_link"/>
-    <origin xyz="0.38 0 0.10" rpy="0 0 0"/>
+    <origin xyz="${camera_x} 0 ${camera_z}" rpy="0 0 0"/>
   </joint>
   <ros2_control name="GazeboSimSystem" type="system">

Commit message: Consolidate Poppy assembly against official reference

File: results/verified/diagnostic/robot.urdf (robot description, URDF)
Before this commit: robot mobile_manipulator, 16 links, 15 joints
Links:
- added link poppy_tool_frame
- link poppy_link_1: geometry collision cylinder length=0.02 radius=0.02; visual mesh filename=file:///home/dryanguasr/proyectos/gazebo-tutorial/gazebo-co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
- link poppy_link_2: geometry collision cylinder length=0.05 radius=0.02; visual mesh filename=file:///home/dryanguasr/proyectos/gazebo-tutorial/gazebo-co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
- link poppy_link_3: geometry collision cylinder length=0.05 radius=0.02; visual mesh filename=file:///home/dryanguasr/proyectos/gazebo-tutorial/gazebo-co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
- link poppy_link_4: geometry collision cylinder length=0.05 radius=0.02; visual mesh filename=file:///home/dryanguasr/proyectos/gazebo-tutorial/gazebo-co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
- link poppy_link_5: geometry collision box size=0.024 0.092 0.006; collision box size=0.036 0.032 0.030
- link poppy_mount_link: geometry collision cylinder length=0.03 radius=0.08; visual mesh filename=file:///home/dryanguasr/proyectos/gazebo-tutorial/gazebo-co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
Joints:
- added joint poppy_tool_frame_joint: type fixed, parent poppy_fixed_tip, child poppy_tool_frame, origin xyz=0 0 0 rpy=0 0 0

File: src/mobile_manipulator/urdf/mobile_manipulator.urdf.xacro (robot description, xacro)
@@ -87,5 +87,9 @@
   <xacro:wheel name="front_right" x="${wheel_x}" y="-${wheel_y}"/>
   <xacro:wheel name="rear_right" x="-${wheel_x}" y="-${wheel_y}"/>
-  <!-- The printed Poppy base and motor m1 body remain fixed to the vehicle. -->
+  <!--
+    Final B3 consolidation: exact visual assembly from the pinned official
+    description. CAD-derived teaching meshes remain under visual/ and are
+    registered in results/verified/mechanical_alignment/alignment_manifest.json.
+  -->
   <link name="poppy_mount_link">
     <inertial>
@@ -95,18 +99,12 @@
     </inertial>
     <visual>
-      <geometry>
-        <mesh filename="file://$(find mobile_manipulator)/meshes/poppy_ergo_jr/visual/poppy_mount.stl"/>
-      </geometry>
-      <material name="PoppyOrange"/>
-    </visual>
-    <visual>
-      <origin xyz="0 0 0.027"/>
-      <geometry><box size="0.024 0.027 0.036"/></geometry>
-      <material name="ServoGray"/>
-    </visual>
-    <collision>
-      <geometry>
-        <mesh filename="file://$(find mobile_manipulator)/meshes/poppy_ergo_jr/collision/poppy_mount_convex.stl"/>
-      </geometry>
+      <origin xyz="0 0 0" rpy="0 0 0"/>
+      <geometry>
+        <mesh filename="file://$(find mobile_manipulator)/meshes/poppy_ergo_jr/official/base.dae"/>
+      </geometry>
+    </visual>
+    <collision>
+      <origin xyz="0 0.038 0.015" rpy="0 0 0"/>
+      <geometry><cylinder length="0.03" radius="0.08"/></geometry>
     </collision>
   </link>
@@ -123,17 +121,12 @@
     </inertial>
     <visual>
-      <geometry>
-        <mesh filename="file://$(find mobile_manipulator)/meshes/poppy_ergo_jr/visual/poppy_link_1.stl"/>
-      </geometry>
-      <material name="PoppyOrange"/>
-    </visual>
-    <visual>
-      <origin xyz="0 0 0.024"/>
-      <geometry><box size="0.024 0.027 0.036"/></geometry>
-      <material name="ServoGray"/>
-    </visual>
-    <collision>
-      <origin xyz="0 0 0.027"/>
-      <geometry><box size="0.042 0.034 0.054"/></geometry>
+      <origin xyz="0 0 0" rpy="0 0 0"/>
+      <geometry>
+        <mesh filename="file://$(find mobile_manipulator)/meshes/poppy_ergo_jr/official/long_U.dae"/>
+      </geometry>
+    </visual>
+    <collision>
+      <origin xyz="0 0 0.01" rpy="0 0 0"/>
+      <geometry><cylinder length="0.02" radius="0.02"/></geometry>
     </collision>
   </link>
@@ -152,17 +145,12 @@
     </inertial>
     <visual>
-      <geometry>
-        <mesh filename="file://$(find mobile_manipulator)/meshes/poppy_ergo_jr/visual/poppy_link_2.stl"/>
-      </geometry>
-      <material name="PoppyOrange"/>
-    </visual>
-    <visual>
-      <origin xyz="0.054 0 0" rpy="0 1.5707963267949 0"/>
-      <geometry><box size="0.027 0.024 0.036"/></geometry>
-      <material name="ServoGray"/>
-    </visual>
-    <collision>
-      <origin xyz="0.0415 0 0"/>
-      <geometry><box size="0.050 0.030 0.040"/></geometry>
+      <origin xyz="0 0 0" rpy="0 1.5707963267949 0"/>
+      <geometry>
+        <mesh filename="file://$(find mobile_manipulator)/meshes/poppy_ergo_jr/official/section_1.dae"/>
+      </geometry>
+    </visual>
+    <collision>
+      <origin xyz="0.025 0 0" rpy="0 1.5707963267949 0"/>
+      <geometry><cylinder length="0.05" radius="0.02"/></geometry>
     </collision>
   </link>
@@ -181,17 +169,12 @@
     </inertial>
     <visual>
-      <geometry>
-        <mesh filename="file://$(find mobile_manipulator)/meshes/poppy_ergo_jr/visual/poppy_link_3.stl"/>
-      </geometry>
-      <material name="PoppyOrange"/>
-    </visual>
-    <visual>
-      <origin xyz="0.045 0 0" rpy="0 1.5707963267949 0"/>
-      <geometry><box size="0.024 0.027 0.036"/></geometry>
-      <material name="ServoGray"/>
-    </visual>
-    <collision>
-      <origin xyz="0.045 0 0"/>
-      <geometry><box size="0.040 0.032 0.036"/></geometry>
+      <origin xyz="0 0 0" rpy="0 1.5707963267949 0"/>
+      <geometry>
+        <mesh filename="file://$(find mobile_manipulator)/meshes/poppy_ergo_jr/official/section_2.dae"/>
+      </geometry>
+    </visual>
+    <collision>
+      <origin xyz="0.025 0 0" rpy="0 1.5707963267949 0"/>
+      <geometry><cylinder length="0.05" radius="0.02"/></geometry>
     </collision>
   </link>
@@ -210,17 +193,12 @@
     </inertial>
     <visual>
-      <geometry>
-        <mesh filename="file://$(find mobile_manipulator)/meshes/poppy_ergo_jr/visual/poppy_link_4.stl"/>
-      </geometry>
-      <material name="PoppyOrange"/>
-    </visual>
-    <visual>
-      <origin xyz="0 -0.048 0" rpy="1.5707963267949 0 0"/>
-      <geometry><box size="0.027 0.024 0.036"/></geometry>
-      <material name="ServoGray"/>
-    </visual>
-    <collision>
-      <origin xyz="0 -0.0415 0"/>
-      <geometry><box size="0.040 0.050 0.030"/></geometry>
+      <origin xyz="0 0 0" rpy="0 3.14159268 0"/>
+      <geometry>
+        <mesh filename="file://$(find mobile_manipulator)/meshes/poppy_ergo_jr/official/section_3.dae"/>
+      </geometry>
+    </visual>
+    <collision>
+      <origin xyz="0 -0.025 0" rpy="1.5707963267949 0 0"/>
+      <geometry><cylinder length="0.05" radius="0.02"/></geometry>
     </collision>
   </link>
@@ -239,13 +217,8 @@
     </inertial>
     <visual>
-      <geometry>
-        <mesh filename="file://$(find mobile_manipulator)/meshes/poppy_ergo_jr/visual/poppy_link_5.stl"/>
-      </geometry>
-      <material name="PoppyOrange"/>
-    </visual>
-    <visual>
       <origin xyz="0 -0.058 0" rpy="0 -1.5707963267949 0"/>
-      <geometry><box size="0.024 0.027 0.036"/></geometry>
-      <material name="ServoGray"/>
+      <geometry>
+        <mesh filename="file://$(find mobile_manipulator)/meshes/poppy_ergo_jr/official/section_4.dae"/>
+      </geometry>
     </visual>
     <collision>
@@ -272,8 +245,8 @@
     </inertial>
     <visual>
-      <geometry>
-        <mesh filename="file://$(find mobile_manipulator)/meshes/poppy_ergo_jr/visual/poppy_link_6.stl"/>
-      </geometry>
-      <material name="PoppyOrange"/>
+      <origin xyz="0 0 0" rpy="0 0 0"/>
+      <geometry>
+        <mesh filename="file://$(find mobile_manipulator)/meshes/poppy_ergo_jr/official/gripper.dae"/>
+      </geometry>
     </visual>
     <collision>
@@ -295,4 +268,10 @@
     <child link="poppy_fixed_tip"/>
     <origin xyz="0 -0.11 0" rpy="-1.5707963267949 0 0"/>
+  </joint>
+  <link name="poppy_tool_frame"/>
+  <joint name="poppy_tool_frame_joint" type="fixed">
+    <parent link="poppy_fixed_tip"/>
+    <child link="poppy_tool_frame"/>
+    <origin xyz="0 0 0" rpy="0 0 0"/>
   </joint>
   <link name="poppy_moving_tip"/>
