Commit message: control: align arm state interfaces with simulation

File: src/mobile_manipulator/urdf/mobile_manipulator.urdf.xacro (robot description, xacro)
@@ -1,5 +1,4 @@
 <?xml version="1.0"?>
 <robot name="mobile_manipulator" xmlns:xacro="http://www.ros.org/wiki/xacro">
-  <xacro:property name="pi" value="3.14159265359"/>
   <xacro:macro name="box" params="name xyz size mass color">
     <link name="${name}"><inertial><mass value="${mass}"/><inertia ixx="0.01" iyy="0.01" izz="0.01" ixy="0" ixz="0" iyz="0"/></inertial><visual><origin xyz="${xyz}"/><geometry><box size="${size}"/></geometry><material name="${color}"/></visual><collision><origin xyz="${xyz}"/><geometry><box size="${size}"/></geometry></collision></link>

Commit message: feat-complete-deterministic-visual-tracking-stack

File: src/mobile_manipulator/urdf/mobile_manipulator.urdf.xacro (robot description, xacro)
@@ -1,4 +1,12 @@
 <?xml version="1.0"?>
 <robot name="mobile_manipulator" xmlns:xacro="http://www.ros.org/wiki/xacro">
+  <material name="SlateGray"><color rgba="0.44 0.50 0.56 1"/></material>
+  <material name="Black"><color rgba="0.04 0.04 0.04 1"/></material>
+  <material name="DarkOrange"><color rgba="1.0 0.35 0.0 1"/></material>
+  <material name="Goldenrod"><color rgba="0.85 0.65 0.13 1"/></material>
+  <material name="Khaki"><color rgba="0.94 0.90 0.55 1"/></material>
+  <material name="LightSteelBlue"><color rgba="0.69 0.77 0.87 1"/></material>
+  <material name="Silver"><color rgba="0.75 0.75 0.75 1"/></material>
+  <material name="Blue"><color rgba="0.1 0.25 0.9 1"/></material>
   <xacro:macro name="box" params="name xyz size mass color">
     <link name="${name}"><inertial><mass value="${mass}"/><inertia ixx="0.01" iyy="0.01" izz="0.01" ixy="0" ixz="0" iyz="0"/></inertial><visual><origin xyz="${xyz}"/><geometry><box size="${size}"/></geometry><material name="${color}"/></visual><collision><origin xyz="${xyz}"/><geometry><box size="${size}"/></geometry></collision></link>

Commit message: feat: add five-lobe tracking demonstration

File: src/mobile_manipulator/urdf/mobile_manipulator.urdf.xacro (robot description, xacro)
@@ -14,5 +14,5 @@
   <xacro:box name="base_link" xyz="0 0 0" size="0.72 0.52 0.16" mass="18" color="SlateGray"/>
   <link name="base_footprint"/><joint name="base_fixed" type="fixed"><parent link="base_footprint"/><child link="base_link"/><origin xyz="0 0 0.16"/></joint>
-  <xacro:macro name="wheel" params="name x y"><link name="${name}_link"><inertial><mass value="1.2"/><inertia ixx="0.006" iyy="0.006" izz="0.01" ixy="0" ixz="0" iyz="0"/></inertial><visual><origin rpy="1.5708 0 0"/><geometry><cylinder radius="0.115" length="0.07"/></geometry><material name="Black"/></visual><collision><origin rpy="1.5708 0 0"/><geometry><cylinder radius="0.115" length="0.07"/></geometry></collision></link><joint name="${name}_joint" type="continuous"><parent link="base_link"/><child link="${name}_link"/><origin xyz="${x} ${y} 0"/><axis xyz="0 1 0"/></joint></xacro:macro>
+  <xacro:macro name="wheel" params="name x y"><link name="${name}_link"><inertial><mass value="1.2"/><inertia ixx="0.006" iyy="0.006" izz="0.01" ixy="0" ixz="0" iyz="0"/></inertial><visual><origin rpy="1.5708 0 0"/><geometry><cylinder radius="0.115" length="0.07"/></geometry><material name="Black"/></visual><collision><origin rpy="1.5708 0 0"/><geometry><cylinder radius="0.115" length="0.07"/></geometry></collision></link><joint name="${name}_joint" type="continuous"><parent link="base_link"/><child link="${name}_link"/><origin xyz="${x} ${y} 0"/><axis xyz="0 1 0"/><limit effort="40" velocity="12.0"/></joint></xacro:macro>
   <xacro:wheel name="front_left" x="0.25" y="0.30"/><xacro:wheel name="rear_left" x="-0.25" y="0.30"/><xacro:wheel name="front_right" x="0.25" y="-0.30"/><xacro:wheel name="rear_right" x="-0.25" y="-0.30"/>
   <xacro:box name="shoulder_link" xyz="0 0 0.13" size="0.18 0.18 0.26" mass="3" color="DarkOrange"/>

Commit message: Implement conditioned Level A pick and place

File: src/mobile_manipulator/urdf/mobile_manipulator.urdf.xacro (robot description, xacro)
@@ -1,4 +1,6 @@
 <?xml version="1.0"?>
 <robot name="mobile_manipulator" xmlns:xacro="http://www.ros.org/wiki/xacro">
+  <xacro:arg name="pick_place_enabled" default="false"/>
+  <xacro:arg name="manipulation_enabled" default="false"/>
   <material name="SlateGray"><color rgba="0.44 0.50 0.56 1"/></material>
   <material name="Black"><color rgba="0.04 0.04 0.04 1"/></material>
@@ -226,7 +228,8 @@
       <geometry><box size="0.036 0.032 0.030"/></geometry>
     </collision>
-    <collision>
-      <origin xyz="0 -0.082 0.0145"/>
-      <geometry><box size="0.024 0.092 0.006"/></geometry>
+    <collision name="poppy_fixed_finger_collision">
+      <!-- Functional contact pad centered on the audited fingertip frame. -->
+      <origin xyz="0 -0.11 0"/>
+      <geometry><sphere radius="0.003"/></geometry>
     </collision>
   </link>
@@ -250,8 +253,8 @@
       </geometry>
     </visual>
-    <collision>
-      <geometry>
-        <mesh filename="file://$(find mobile_manipulator)/meshes/poppy_ergo_jr/collision/poppy_link_6_convex.stl"/>
-      </geometry>
+    <collision name="poppy_moving_finger_collision">
+      <!-- Functional contact pad centered on the audited fingertip frame. -->
+      <origin xyz="0 -0.052 0"/>
+      <geometry><sphere radius="0.003"/></geometry>
     </collision>
   </link>
@@ -274,4 +277,15 @@
     <child link="poppy_tool_frame"/>
     <origin xyz="0 0 0" rpy="0 0 0"/>
+  </joint>
+  <!--
+    The validated tool frame remains on the fixed fingertip.  At m6=0.60 rad,
+    this grasp frame is the midpoint between the two audited fingertip frames;
+    it does not redefine or move poppy_tool_frame.
+  -->
+  <link name="poppy_grasp_frame"/>
+  <joint name="poppy_grasp_frame_joint" type="fixed">
+    <parent link="poppy_tool_frame"/>
+    <child link="poppy_grasp_frame"/>
+    <origin xyz="0 0.0147 0.00455" rpy="0 0 0"/>
   </joint>
   <link name="poppy_moving_tip"/>
@@ -358,5 +372,27 @@
     <plugin filename="gz_ros2_control-system" name="gz_ros2_control::GazeboSimROS2ControlPlugin">
       <parameters>$(find mobile_manipulator)/config/controllers.yaml</parameters>
+      <xacro:if value="$(arg manipulation_enabled)">
+        <position_proportional_gain>2.0</position_proportional_gain>
+      </xacro:if>
     </plugin>
   </gazebo>
+  <xacro:if value="$(arg pick_place_enabled)">
+    <!--
+      Gazebo Sim 8 DetachableJoint is simulator assistance, not physical grasp.
+      The plugin is configured before pick_object is spawned, detached during
+      RESET, and commanded only by the bilateral-contact gate.
+    -->
+    <gazebo>
+      <plugin filename="gz-sim-detachable-joint-system"
+              name="gz::sim::systems::DetachableJoint">
+        <parent_link>poppy_link_5</parent_link>
+        <child_model>pick_object</child_model>
+        <child_link>object_link</child_link>
+        <detach_topic>/pick_object/detach</detach_topic>
+        <attach_topic>/pick_object/attach</attach_topic>
+        <output_topic>/pick_object/joint_state</output_topic>
+        <suppress_child_warning>true</suppress_child_warning>
+      </plugin>
+    </gazebo>
+  </xacro:if>
 </robot>

Commit message: Preserve baseline gripper collisions outside manipulation

File: src/mobile_manipulator/urdf/mobile_manipulator.urdf.xacro (robot description, xacro)
@@ -228,9 +228,17 @@
       <geometry><box size="0.036 0.032 0.030"/></geometry>
     </collision>
-    <collision name="poppy_fixed_finger_collision">
-      <!-- Functional contact pad centered on the audited fingertip frame. -->
-      <origin xyz="0 -0.11 0"/>
-      <geometry><sphere radius="0.003"/></geometry>
-    </collision>
+    <xacro:unless value="$(arg manipulation_enabled)">
+      <collision>
+        <origin xyz="0 -0.082 0.0145"/>
+        <geometry><box size="0.024 0.092 0.006"/></geometry>
+      </collision>
+    </xacro:unless>
+    <xacro:if value="$(arg manipulation_enabled)">
+      <collision name="poppy_fixed_finger_collision">
+        <!-- Functional contact pad centered on the audited fingertip frame. -->
+        <origin xyz="0 -0.11 0"/>
+        <geometry><sphere radius="0.003"/></geometry>
+      </collision>
+    </xacro:if>
   </link>
   <joint name="poppy_m5_joint" type="revolute">
@@ -253,9 +261,18 @@
       </geometry>
     </visual>
-    <collision name="poppy_moving_finger_collision">
-      <!-- Functional contact pad centered on the audited fingertip frame. -->
-      <origin xyz="0 -0.052 0"/>
-      <geometry><sphere radius="0.003"/></geometry>
-    </collision>
+    <xacro:unless value="$(arg manipulation_enabled)">
+      <collision>
+        <geometry>
+          <mesh filename="file://$(find mobile_manipulator)/meshes/poppy_ergo_jr/collision/poppy_link_6_convex.stl"/>
+        </geometry>
+      </collision>
+    </xacro:unless>
+    <xacro:if value="$(arg manipulation_enabled)">
+      <collision name="poppy_moving_finger_collision">
+        <!-- Functional contact pad centered on the audited fingertip frame. -->
+        <origin xyz="0 -0.052 0"/>
+        <geometry><sphere radius="0.003"/></geometry>
+      </collision>
+    </xacro:if>
   </link>
   <joint name="poppy_m6_joint" type="revolute">

Commit message: fix: correct physical grasp and Gazebo gripper assembly
Align contact geometry and enforce physical retention checks. Bake repeated CAD instances for correct Gazebo rendering and add inspection colors. Include regression tests, verified runs, and 60 fps capture evidence.

File: src/mobile_manipulator/urdf/mobile_manipulator.urdf.xacro (robot description, xacro)
@@ -90,6 +90,7 @@
   <xacro:wheel name="rear_right" x="-${wheel_x}" y="-${wheel_y}"/>
   <!--
-    Final B3 consolidation: exact visual assembly from the pinned official
-    description. CAD-derived teaching meshes remain under visual/ and are
+    Gazebo-compatible visual assembly from the pinned official description:
+    instance transforms are baked; original files remain under official/.
+    CAD-derived teaching meshes remain under visual/ and are
     registered in results/verified/mechanical_alignment/alignment_manifest.json.
   -->
@@ -103,5 +104,5 @@
       <origin xyz="0 0 0" rpy="0 0 0"/>
       <geometry>
-        <mesh filename="file://$(find mobile_manipulator)/meshes/poppy_ergo_jr/official/base.dae"/>
+        <mesh filename="file://$(find mobile_manipulator)/meshes/poppy_ergo_jr/gazebo_inspection/base.dae"/>
       </geometry>
     </visual>
@@ -125,5 +126,5 @@
       <origin xyz="0 0 0" rpy="0 0 0"/>
       <geometry>
-        <mesh filename="file://$(find mobile_manipulator)/meshes/poppy_ergo_jr/official/long_U.dae"/>
+        <mesh filename="file://$(find mobile_manipulator)/meshes/poppy_ergo_jr/gazebo_inspection/long_U.dae"/>
       </geometry>
     </visual>
@@ -149,5 +150,5 @@
       <origin xyz="0 0 0" rpy="0 1.5707963267949 0"/>
       <geometry>
-        <mesh filename="file://$(find mobile_manipulator)/meshes/poppy_ergo_jr/official/section_1.dae"/>
+        <mesh filename="file://$(find mobile_manipulator)/meshes/poppy_ergo_jr/gazebo_inspection/section_1.dae"/>
       </geometry>
     </visual>
@@ -173,5 +174,5 @@
       <origin xyz="0 0 0" rpy="0 1.5707963267949 0"/>
       <geometry>
-        <mesh filename="file://$(find mobile_manipulator)/meshes/poppy_ergo_jr/official/section_2.dae"/>
+        <mesh filename="file://$(find mobile_manipulator)/meshes/poppy_ergo_jr/gazebo_inspection/section_2.dae"/>
       </geometry>
     </visual>
@@ -197,5 +198,5 @@
       <origin xyz="0 0 0" rpy="0 3.14159268 0"/>
       <geometry>
-        <mesh filename="file://$(find mobile_manipulator)/meshes/poppy_ergo_jr/official/section_3.dae"/>
+        <mesh filename="file://$(find mobile_manipulator)/meshes/poppy_ergo_jr/gazebo_inspection/section_3.dae"/>
       </geometry>
     </visual>
@@ -221,5 +222,5 @@
       <origin xyz="0 -0.058 0" rpy="0 -1.5707963267949 0"/>
       <geometry>
-        <mesh filename="file://$(find mobile_manipulator)/meshes/poppy_ergo_jr/official/section_4.dae"/>
+        <mesh filename="file://$(find mobile_manipulator)/meshes/poppy_ergo_jr/gazebo_inspection/section_4.dae"/>
       </geometry>
     </visual>
@@ -236,7 +237,7 @@
     <xacro:if value="$(arg manipulation_enabled)">
       <collision name="poppy_fixed_finger_collision">
-        <!-- Functional contact pad centered on the audited fingertip frame. -->
-        <origin xyz="0 -0.11 0"/>
-        <geometry><sphere radius="0.003"/></geometry>
+        <!-- Inner face z=14 mm matches the official distal CAD plate. -->
+        <origin xyz="0 -0.110 0.01555"/>
+        <geometry><box size="0.024 0.030 0.0031"/></geometry>
       </collision>
     </xacro:if>
@@ -258,5 +259,5 @@
       <origin xyz="0 0 0" rpy="0 0 0"/>
       <geometry>
-        <mesh filename="file://$(find mobile_manipulator)/meshes/poppy_ergo_jr/official/gripper.dae"/>
+        <mesh filename="file://$(find mobile_manipulator)/meshes/poppy_ergo_jr/gazebo_inspection/gripper.dae"/>
       </geometry>
     </visual>
@@ -270,7 +271,6 @@
     <xacro:if value="$(arg manipulation_enabled)">
       <collision name="poppy_moving_finger_collision">
-        <!-- Functional contact pad centered on the audited fingertip frame. -->
-        <origin xyz="0 -0.052 0"/>
-        <geometry><sphere radius="0.003"/></geometry>
+        <origin xyz="-0.01555 -0.052 0.0001"/>
+        <geometry><box size="0.0031 0.030 0.024"/></geometry>
       </collision>
     </xacro:if>
@@ -296,7 +296,7 @@
   </joint>
   <!--
-    The validated tool frame remains on the fixed fingertip.  At m6=0.60 rad,
-    this grasp frame is the midpoint between the two audited fingertip frames;
-    it does not redefine or move poppy_tool_frame.
+    The historical tool/tip frames are retained for tracking compatibility.
+    Actual contact frames lie on the visible inner CAD surfaces. The grasp
+    center fits a 30 mm cylinder at m6 approximately 0.04 rad.
   -->
   <link name="poppy_grasp_frame"/>
@@ -304,5 +304,5 @@
     <parent link="poppy_tool_frame"/>
     <child link="poppy_grasp_frame"/>
-    <origin xyz="0 0.0147 0.00455" rpy="0 0 0"/>
+    <origin xyz="0 0.0015 0" rpy="0 0 0"/>
   </joint>
   <link name="poppy_moving_tip"/>
@@ -311,4 +311,16 @@
     <child link="poppy_moving_tip"/>
     <origin xyz="0 -0.052 0" rpy="-1.5707963267949 0 0"/>
+  </joint>
+  <link name="poppy_fixed_contact"/>
+  <joint name="poppy_fixed_contact_joint" type="fixed">
+    <parent link="poppy_link_5"/>
+    <child link="poppy_fixed_contact"/>
+    <origin xyz="0 -0.110 0.014"/>
+  </joint>
+  <link name="poppy_moving_contact"/>
+  <joint name="poppy_moving_contact_joint" type="fixed">
+    <parent link="poppy_link_6"/>
+    <child link="poppy_moving_contact"/>
+    <origin xyz="-0.014 -0.052 0.0001"/>
   </joint>
   <!-- The tracking camera stays on the vehicle front to preserve the A/B task. -->
